File: kicad/stereo_sonic_beast.kicad_pcb (KiCad board)
At the start: 2 copper layers, 94.9 x 60 mm, 77 parts, among them J1 DB25_Male_MountingHoles, J2 Barrel_Jack, J3 SJ1-3535NG, SW1 SW_DIP_x03, SW2 SW_DIP_x03, U1 ATF22V10CQZ-20PU, U2 ATF22V10CQZ-20PU

Commit message: PDF file for schema added.
Other:
- board text added: "Stereo Sonic Beast Rev 1.4 by Damouze 2021."
- board text removed: "Stereo Sonic Beast Rev 1.2 by Damouze 2021."
